File: Payload_PCB/payload_bhi160B.kicad_sch (KiCad schematic)
At the start: 9 parts, among them U7 BHI160B

Commit message: Minor changes and corrections
Parts:
- renumbered C1 to C12, C2 to C13, C3 to C14, C4 to C15, R1 to R45, R2 to R46, R3 to R47, R4 to R48, U7 to U8
Changed lines of the file:
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@@
   (symbol (lib_id "Device:R_Small") (at 168.275 105.41 90) (unit 1)
     (in_bom yes) (on_board yes) (dnp no)
-    (property "Reference" "R4" (at 168.275 103.505 90)
+    (property "Reference" "R48" (at 168.275 103.505 90)
       (effects (font (size 1.27 1.27)))
     )
@@
       (project "Payload_PCB"
         (path "/5c4f9a68-5778-4223-b18a-2e31db8d7d40/d52ba4fa-6dae-452c-85f1-a72652abf275/303d15aa-29fe-42a5-a6a1-f7f24dc6bce2"
+          (reference "R48") (unit 1)
+        )
+      )
+      (project "Payload_Sensors"
+        (path "/be15da96-a8ba-4b41-94e6-4486ed8c384e/303d15aa-29fe-42a5-a6a1-f7f24dc6bce2"
           (reference "R4") (unit 1)
         )
       )
-      (project "Payload_Sensors"
-        (path "/be15da96-a8ba-4b41-94e6-4486ed8c384e/303d15aa-29fe-42a5-a6a1-f7f24dc6bce2"
-          (reference "R4") (unit 1)
-        )
-      )
     )
   )
   (symbol (lib_id "Device:C_Small") (at 198.12 97.79 270) (mirror x) (unit 1)
     (in_bom yes) (on_board yes) (dnp no)
-    (property "Reference" "C4" (at 198.12 95.25 90)
+    (property "Reference" "C15" (at 198.12 95.25 90)
       (effects (font (size 1.27 1.27)))
     )
@@
       (project "Payload_PCB"
         (path "/5c4f9a68-5778-4223-b18a-2e31db8d7d40/d52ba4fa-6dae-452c-85f1-a72652abf275/303d15aa-29fe-42a5-a6a1-f7f24dc6bce2"
+          (reference "C15") (unit 1)
+        )
+      )
+      (project "Payload_Sensors"
+        (path "/be15da96-a8ba-4b41-94e6-4486ed8c384e/303d15aa-29fe-42a5-a6a1-f7f24dc6bce2"
           (reference "C4") (unit 1)
         )
       )
-      (project "Payload_Sensors"
-        (path "/be15da96-a8ba-4b41-94e6-4486ed8c384e/303d15aa-29fe-42a5-a6a1-f7f24dc6bce2"
-          (reference "C4") (unit 1)
-        )
-      )
     )
   )
   (symbol (lib_id "Device:C_Small") (at 192.405 93.98 270) (mirror x) (unit 1)
     (in_bom yes) (on_board yes) (dnp no)
-    (property "Reference" "C3" (at 192.405 91.44 90)
+    (property "Reference" "C14" (at 192.405 91.44 90)
       (effects (font (size 1.27 1.27)))
     )
@@
       (project "Payload_PCB"
         (path "/5c4f9a68-5778-4223-b18a-2e31db8d7d40/d52ba4fa-6dae-452c-85f1-a72652abf275/303d15aa-29fe-42a5-a6a1-f7f24dc6bce2"
+          (reference "C14") (unit 1)
+        )
+      )
+      (project "Payload_Sensors"
+        (path "/be15da96-a8ba-4b41-94e6-4486ed8c384e/303d15aa-29fe-42a5-a6a1-f7f24dc6bce2"
           (reference "C3") (unit 1)
         )
       )
-      (project "Payload_Sensors"
-        (path "/be15da96-a8ba-4b41-94e6-4486ed8c384e/303d15aa-29fe-42a5-a6a1-f7f24dc6bce2"
-          (reference "C3") (unit 1)
-        )
-      )
     )
   )
   (symbol (lib_id "Device:C_Small") (at 187.96 90.17 270) (unit 1)
     (in_bom yes) (on_board yes) (dnp no)
-    (property "Reference" "C2" (at 187.96 87.63 90)
+    (property "Reference" "C13" (at 187.96 87.63 90)
       (effects (font (size 1.27 1.27)))
     )
@@
       (project "Payload_PCB"
         (path "/5c4f9a68-5778-4223-b18a-2e31db8d7d40/d52ba4fa-6dae-452c-85f1-a72652abf275/303d15aa-29fe-42a5-a6a1-f7f24dc6bce2"
-          (reference "C2") (unit 1)
+          (reference "C13") (unit 1)
         )
       )
@@
   (symbol (lib_name "BHI160B_1") (lib_id "BHI160B:BHI160B") (at 139.7 107.95 0) (unit 1)
     (in_bom yes) (on_board yes) (dnp no) (fields_autoplaced)
-    (property "Reference" "U7" (at 139.7 82.55 0)
+    (property "Reference" "U8" (at 139.7 82.55 0)
       (effects (font (size 1.27 1.27)))
     )
@@
       (project "Payload_PCB"
         (path "/5c4f9a68-5778-4223-b18a-2e31db8d7d40/d52ba4fa-6dae-452c-85f1-a72652abf275/303d15aa-29fe-42a5-a6a1-f7f24dc6bce2"
+          (reference "U8") (unit 1)
+        )
+      )
+      (project "Payload_Sensors"
+        (path "/be15da96-a8ba-4b41-94e6-4486ed8c384e/303d15aa-29fe-42a5-a6a1-f7f24dc6bce2"
           (reference "U7") (unit 1)
         )
       )
-      (project "Payload_Sensors"
-        (path "/be15da96-a8ba-4b41-94e6-4486ed8c384e/303d15aa-29fe-42a5-a6a1-f7f24dc6bce2"
-          (reference "U7") (unit 1)
-        )
-      )
     )
   )
   (symbol (lib_id "Device:C_Small") (at 182.88 86.36 270) (unit 1)
     (in_bom yes) (on_board yes) (dnp no)
-    (property "Reference" "C1" (at 182.88 83.82 90)
+    (property "Reference" "C12" (at 182.88 83.82 90)
       (effects (font (size 1.27 1.27)))
     )
@@
       (project "Payload_PCB"
         (path "/5c4f9a68-5778-4223-b18a-2e31db8d7d40/d52ba4fa-6dae-452c-85f1-a72652abf275/303d15aa-29fe-42a5-a6a1-f7f24dc6bce2"
+          (reference "C12") (unit 1)
+        )
+      )
+      (project "Payload_Sensors"
+        (path "/be15da96-a8ba-4b41-94e6-4486ed8c384e/303d15aa-29fe-42a5-a6a1-f7f24dc6bce2"
           (reference "C1") (unit 1)
         )
       )
-      (project "Payload_Sensors"
-        (path "/be15da96-a8ba-4b41-94e6-4486ed8c384e/303d15aa-29fe-42a5-a6a1-f7f24dc6bce2"
-          (reference "C1") (unit 1)
-        )
-      )
     )
   )
   (symbol (lib_id "Device:R_Small") (at 140.335 64.77 90) (unit 1)
     (in_bom yes) (on_board yes) (dnp no)
-    (property "Reference" "R1" (at 140.335 62.865 90)
+    (property "Reference" "R45" (at 140.335 62.865 90)
       (effects (font (size 1.27 1.27)))
     )
@@
       (project "Payload_PCB"
         (path "/5c4f9a68-5778-4223-b18a-2e31db8d7d40/d52ba4fa-6dae-452c-85f1-a72652abf275/303d15aa-29fe-42a5-a6a1-f7f24dc6bce2"
+          (reference "R45") (unit 1)
+        )
+      )
+      (project "Payload_Sensors"
+        (path "/be15da96-a8ba-4b41-94e6-4486ed8c384e/303d15aa-29fe-42a5-a6a1-f7f24dc6bce2"
           (reference "R1") (unit 1)
         )
       )
-      (project "Payload_Sensors"
-        (path "/be15da96-a8ba-4b41-94e6-4486ed8c384e/303d15aa-29fe-42a5-a6a1-f7f24dc6bce2"
-          (reference "R1") (unit 1)
-        )
-      )
     )
   )
   (symbol (lib_id "Device:R_Small") (at 140.335 70.485 90) (unit 1)
     (in_bom yes) (on_board yes) (dnp no)
-    (property "Reference" "R2" (at 140.335 68.58 90)
+    (property "Reference" "R46" (at 140.335 68.58 90)
       (effects (font (size 1.27 1.27)))
     )
@@
       (project "Payload_PCB"
         (path "/5c4f9a68-5778-4223-b18a-2e31db8d7d40/d52ba4fa-6dae-452c-85f1-a72652abf275/303d15aa-29fe-42a5-a6a1-f7f24dc6bce2"
+          (reference "R46") (unit 1)
+        )
+      )
+      (project "Payload_Sensors"
+        (path "/be15da96-a8ba-4b41-94e6-4486ed8c384e/303d15aa-29fe-42a5-a6a1-f7f24dc6bce2"
           (reference "R2") (unit 1)
         )
       )
-      (project "Payload_Sensors"
-        (path "/be15da96-a8ba-4b41-94e6-4486ed8c384e/303d15aa-29fe-42a5-a6a1-f7f24dc6bce2"
-          (reference "R2") (unit 1)
-        )
-      )
     )
   )
   (symbol (lib_id "Device:R_Small") (at 161.925 102.87 90) (unit 1)
     (in_bom yes) (on_board yes) (dnp no)
-    (property "Reference" "R3" (at 161.925 100.965 90)
+    (property "Reference" "R47" (at 161.925 100.965 90)
       (effects (font (size 1.27 1.27)))
     )
@@
       (project "Payload_PCB"
         (path "/5c4f9a68-5778-4223-b18a-2e31db8d7d40/d52ba4fa-6dae-452c-85f1-a72652abf275/303d15aa-29fe-42a5-a6a1-f7f24dc6bce2"
-          (reference "R3") (unit 1)
-        )
-      )
+          (reference "R47") (unit 1)
+        )
+      )
