File: Payload_PCB/payload_bmp390.kicad_sch (KiCad schematic)
At the start: 5 parts, among them IC1 BMP390

Commit message: Adjust page size
Other:
- moved on the sheet: C14, C15, IC1, R45, R46

Commit message: Added some actual parts
Parts:
- C15: value C_Small -> 100nF
Changed lines of the file:
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@@
       (effects (font (size 1.27 1.27)) (justify left))
     )
-    (property "Value" "C_Small" (at 139.7 66.6813 0)
+    (property "Value" "100nF" (at 139.7 66.6813 0)
       (effects (font (size 1.27 1.27)) (justify left))
     )
