File: Payload_PCB/Payload_PCB.kicad_sch (KiCad schematic)
At the start: 25 parts, among them IC1 BU4S584G2-TL, J1 43650-0315, J2 43650-0315, J3 43650-0315, J4 43650-0315, J5 43650-0400, Q3 PMOS, U10 TPS61253YFFR, U2 TPS61253YFFR

Commit message: Todo notes after review
Parts:
- removed D4: RB511VM-30TE-17, footprints:RB511VM30TE17, symbol RB511VM-30TE-17:RB511VM-30TE-17
- added R45: 1kOhm, symbol Device:R
Connections:
- net VDD: now also IC1.5 (VDD), R45.1
- net Schmitt_VCC: no longer names the net of cutoff_plug1.1
- net Schmitt_VCC: now also R45.2; no longer IC1.5 (VDD)
Other:
- note added: "BMS_VIN woher?"
- note added: "Mit Avionics integrieren: ein "Plug" als connector"
- note added: "Nochmal Boost Conv. anschauen Layout wie?"
- note added: "RS Flag direkt dran"
- note added: "Spule vllt"
- note added: "Statt VDD Batteriespannung rausführen"
- note added: "TODO: Zwischen MOSI, CLK, und MISO GND"
Changed lines of the file:
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@@
   (junction (at 173.355 90.17) (diameter 0) (color 0 0 0 0)
   )
-  (junction (at 39.37 220.98) (diameter 0) (color 0 0 0 0)
-  )
   (junction (at 260.35 235.585) (diameter 0) (color 0 0 0 0)
   )
@@
     (stroke (width 0) (type default))
   )
-  (polyline (pts (xy 12.065 230.505) (xy 109.22 230.505))
+  (polyline (pts (xy 12.065 233.045) (xy 109.22 233.045))
     (stroke (width 0) (type dash))
   )
@@
     (stroke (width 0) (type default))
   )
+  (wire (pts (xy 33.655 220.98) (xy 47.625 220.98))
+    (stroke (width 0) (type default))
+  )
   (polyline (pts (xy 180.975 200.66) (xy 180.975 285.115))
     (stroke (width 0) (type default))
@@
     (stroke (width 0) (type default))
   )
-  (wire (pts (xy 39.37 220.98) (xy 47.625 220.98))
-    (stroke (width 0) (type default))
-  )
   (wire (pts (xy 369.57 231.775) (xy 370.84 231.775))
     (stroke (width 0) (type default))
@@
     (stroke (width 0) (type default))
   )
-  (wire (pts (xy 39.37 220.98) (xy 39.37 210.82))
-    (stroke (width 0) (type default))
-  )
   (wire (pts (xy 173.99 110.49) (xy 173.99 113.03))
     (stroke (width 0) (type default))
@@
     (stroke (width 0) (type default))
   )
-  (wire (pts (xy 86.36 220.98) (xy 93.345 220.98))
+  (wire (pts (xy 86.36 220.98) (xy 96.52 220.98))
     (stroke (width 0) (type default))
   )
@@
     (stroke (width 0) (type default))
   )
-  (wire (pts (xy 86.36 226.06) (xy 88.9 226.06))
+  (wire (pts (xy 86.36 226.06) (xy 80.645 226.06))
     (stroke (width 0) (type default))
   )
@@
     (stroke (width 0) (type default))
   )
-  (wire (pts (xy 33.655 220.98) (xy 39.37 220.98))
-    (stroke (width 0) (type default))
-  )
   (wire (pts (xy 183.515 99.06) (xy 183.515 100.33))
     (stroke (width 0) (type default))
@@
     (stroke (width 0) (type default))
   )
-  (wire (pts (xy 29.21 210.82) (xy 39.37 210.82))
-    (stroke (width 0) (type default))
-  )
   (wire (pts (xy 63.5 209.55) (xy 71.12 209.55))
     (stroke (width 0) (type default))
@@
     (effects (font (size 1.27 1.27)) (justify left bottom))
   )
+  (text "Statt VDD Batteriespannung rausführen" (at 12.7 226.06 0)
+    (effects (font (size 1.27 1.27)) (justify left bottom))
+  )
   (text "S GND\n" (at 218.44 167.64 0)
     (effects (font (size 1.27 1.27)) (justify left bottom))
@@
   )
   (text "GND (R)" (at 23.495 56.515 0)
+    (effects (font (size 1.27 1.27)) (justify left bottom))
+  )
+  (text "TODO: Zwischen MOSI, CLK, und MISO GND" (at 114.3 140.97 0)
     (effects (font (size 1.27 1.27)) (justify left bottom))
   )
@@
     (effects (font (size 0.635 0.635)) (justify left bottom))
   )
+  (text "RS Flag direkt dran" (at 41.91 208.28 0)
+    (effects (font (size 1.27 1.27)) (justify left bottom))
+  )
+  (text "Mit Avionics integrieren: ein \"Plug\" als connector"
+    (at 12.7 204.47 0)
+    (effects (font (size 1.27 1.27)) (justify left bottom))
+  )
+  (text "BMS_VIN woher?" (at 17.145 139.7 0)
+    (effects (font (size 1.27 1.27)) (justify left bottom))
+  )
   (text "Schmitt Inverter" (at 55.245 264.16 0)
     (effects (font (size 1.27 1.27)) (justify left bottom))
@@
     (effects (font (size 1.27 1.27)) (justify left bottom))
   )
+  (text "Spule vllt" (at 222.25 51.435 0)
+    (effects (font (size 1.27 1.27)) (justify left bottom))
+  )
   (text "3.3V" (at 137.16 163.83 0)
     (effects (font (size 1.27 1.27)) (justify left bottom))
@@
   )
   (text "Radio Silence Main Part\n" (at 73.66 281.94 0)
+    (effects (font (size 1.27 1.27)) (justify left bottom))
+  )
+  (text "Nochmal Boost Conv. anschauen\nLayout wie?" (at 214.63 21.59 0)
     (effects (font (size 1.27 1.27)) (justify left bottom))
   )
@@
     )
   )
-  (global_label "Schmitt_VCC" (shape output) (at 29.21 210.82 180) (fields_autoplaced)
-    (effects (font (size 1.27 1.27)) (justify right))
-    (property "Intersheetrefs" "${INTERSHEET_REFS}" (at 14.432 210.82 0)
-      (effects (font (size 1.27 1.27)) (justify right) hide)
-    )
-  )
   (global_label "SDA" (shape input) (at 214.63 226.06 180) (fields_autoplaced)
     (effects (font (size 1.27 1.27)) (justify right))
@@
     )
   )
-  (global_label "Schmitt_VCC" (shape input) (at 75.565 256.54 0) (fields_autoplaced)
-    (effects (font (size 1.27 1.27)) (justify left))
-    (property "Intersheetrefs" "${INTERSHEET_REFS}" (at 90.343 256.54 0)
+  (global_label "VDD" (shape input) (at 75.565 256.54 0) (fields_autoplaced)
+    (effects (font (size 1.27 1.27)) (justify left))
+    (property "Intersheetrefs" "${INTERSHEET_REFS}" (at 82.1788 256.54 0)
       (effects (font (size 1.27 1.27)) (justify left) hide)
     )
@@
     )
   )
-  (global_label "Short{slash}Discharge" (shape output) (at 88.9 226.06 0) (fields_autoplaced)
-    (effects (font (size 1.27 1.27)) (justify left))
-    (property "Intersheetrefs" "${INTERSHEET_REFS}" (at 107.5484 226.06 0)
-      (effects (font (size 1.27 1.27)) (justify left) hide)
-    )
-  )
-  (global_label "RS_Gate" (shape output) (at 93.345 220.98 0) (fields_autoplaced)
-    (effects (font (size 1.27 1.27)) (justify left))
-    (property "Intersheetrefs" "${INTERSHEET_REFS}" (at 104.0106 220.98 0)
+  (global_label "Short{slash}Discharge" (shape output) (at 80.645 226.06 180) (fields_autoplaced)
+    (effects (font (size 1.27 1.27)) (justify right))
+    (property "Intersheetrefs" "${INTERSHEET_REFS}" (at 61.9966 226.06 0)
+      (effects (font (size 1.27 1.27)) (justify right) hide)
+    )
+  )
+  (global_label "RS_Gate" (shape output) (at 96.52 220.98 0) (fields_autoplaced)
+    (effects (font (size 1.27 1.27)) (justify left))
+    (property "Intersheetrefs" "${INTERSHEET_REFS}" (at 107.1856 220.98 0)
       (effects (font (size 1.27 1.27)) (justify left) hide)
     )
@@
     )
   )
+  (symbol (lib_id "Device:R") (at 29.845 220.98 90) (unit 1)
+    (in_bom yes) (on_board yes) (dnp no) (fields_autoplaced)
+    (property "Reference" "R45" (at 29.845 214.63 90)
+      (effects (font (size 1.27 1.27)))
+    )
+    (property "Value" "1kOhm" (at 29.845 217.17 90)
+      (effects (font (size 1.27 1.27)))
+    )
+    (property "Footprint" "" (at 29.845 222.758 90)
+      (effects (font (size 1.27 1.27)) hide)
+    )
+    (property "Datasheet" "~" (at 29.845 220.98 0)
+      (effects (font (size 1.27 1.27)) hide)
+    )
+    (pin "1")
+    (pin "2")
+    (instances
+      (project "Payload_PCB"
+        (path "/5c4f9a68-5778-4223-b18a-2e31db8d7d40"
+          (reference "R45") (unit 1)
+        )
+      )
+    )
+  )
   (symbol (lib_id "Simulation_SPICE:PMOS") (at 206.375 54.61 270) (mirror x) (unit 1)
     (in_bom yes) (on_board yes) (dnp no)
@@
         )
       )
-    )
-  )
-  (symbol (lib_id "RB511VM-30TE-17:RB511VM-30TE-17") (at 33.655 220.98 180) (unit 1)
-    (in_bom yes) (on_board yes) (dnp no) (fields_autoplaced)
-    (property "Reference" "D4" (at 29.845 215.265 0)
-      (effects (font (size 1.27 1.27)))
-    )
-    (property "Value" "RB511VM-30TE-17" (at 29.845 217.805 0)
-      (effects (font (size 1.27 1.27)))
-    )
-    (property "Footprint" "footprints:RB511VM30TE17" (at 22.225 123.52 0)
-      (effects (font (size 1.27 1.27)) (justify left top) hide)
-    )
-    (property "Datasheet" "https://datasheet.datasheetarchive.com/originals/distributors/Datasheets_SAMA/104678791d62a70c3f3b75cb640f2c08.pdf" (at 22.225 23.52 0)
-      (effects (font (size 1.27 1.27)) (justify left top) hide)
-    )
-    (property "Height" "0.9" (at 22.225 -176.48 0)
-      (effects (font (size 1.27 1.27)) (justify left top) hide)
-    )
-    (property "Mouser Part Number" "755-RB511VM-30TE-17" (at 22.225 -276.48 0)
-      (effects (font (size 1.27 1.27)) (justify left top) hide)
-    )
-    (property "Mouser Price/Stock" "https://www.mouser.co.uk/ProductDetail/ROHM-Semiconductor/RB511VM-30TE-17?qs=4v%252BiZTmLVHHI3%252BFheXsKTQ%3D%3D" (at 22.225 -376.48 0)
-      (effects (font (size 1.27 1.27)) (justify left top) hide)
-    )
-    (property "Manufacturer_Name" "ROHM Semiconductor" (at 22.225 -476.48 0)
-      (effects (font (size 1.27 1.27)) (justify left top) hide)
-    )
-    (property "Manufacturer_Part_Number" "RB511VM-30TE-17" (at 22.225 -576.48 0)
-      (effects (font (size 1.27 1.27)) (justify left top) hide)
-    )
-    (pin "1")
-    (pin "2")
-    (instances
-      (project "Payload_PCB"
-        (path "/5c4f9a68-5778-4223-b18a-2e31db8d7d40"
-          (reference "D4") (unit 1)
-        )
-      )
