File: Payload_PCB/Payload_PCB.kicad_sch (KiCad schematic)
At the start: 25 parts, among them IC1 BU4S584G2-TL, J1 43650-0315, J2 43650-0315, J3 43650-0315, J4 43650-0315, J5 43650-0400, Q3 PMOS, U10 TPS61253YFFR, U2 TPS61253YFFR

Commit message: first parts layout
Parts:
- removed IC1: BU4S584G2-TL, footprints:SOT95P280X125-5N, symbol BU4S584G2-TL:BU4S584G2-TL
- removed R1: 5k, symbol Device:R
- removed R2: 10k, symbol Device:R
Connections:
- net Schmitt_Out is gone; now on net RS_Flag: D1.2 (A)
- net VDD: no longer R45.1
Other:
- sheet Charge_MCP73834_1 ports: added BAT_VDD; removed none
- note added: "Connector"
- note removed: "Radio Silence Main Part"
- note removed: "Schmitt Inverter"
- note removed: "Statt VDD Batteriespannung rausführen"
- moved on the sheet: C1, C18, C2, D1, D2, D5, L1, L2, LED_Conn1, Q3, R4, R45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
