File: Payload_PCB/Payload_TC_MC.kicad_sch (KiCad schematic)
At the start: 9 parts, among them U4 MCP9601-E/MX

Commit message: Minor changes and corrections
Parts:
- renumbered C2 to C7, D3 to D10, D4 to D11, R3 to R25, R2 to R26, R1 to R27, R17 to R28, U4 to U3
Connections:
- net VDD renamed VIN_TC

Commit message: Added heating pad, adjustment of page sizes
Other:
- moved on the sheet: C7, D10, D11, R25, R26, R27, R28, TC1, U3

Commit message: Added some actual parts
Parts:
- removed D10, D11: D_Schottky_Small, symbol Device:D_Schottky_Small
- added R79: 10kOhm, symbol Device:R
- R28: value R -> 10kOhm
Connections:
- net GND: now also R79.2
- net OCALERT: now also U3.9 (OCALERT), R79.1; no longer R28.1
- net SCALERT: now reaches U3.7 (SCALERT)
- net SCALERT: now also R28.1
Other:
- company: (none) -> SpaceTeam Aachen
- title: (none) -> Thermocouple Microchip
- moved on the sheet: R26, R27, R28, TC1

Commit message: Change to actual real parts
Changed lines of the file:
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@@
     )
   )
-  (global_label "GND" (shape input) (at 104.775 81.28 0) (fields_autoplaced)
+  (global_label "GND" (shape output) (at 104.775 81.28 0) (fields_autoplaced)
     (effects (font (size 1.27 1.27)) (justify left))
     (property "Intersheetrefs" "${INTERSHEET_REFS}" (at 111.6307 81.28 0)
@@
     )
   )
-  (global_label "GND" (shape input) (at 53.975 71.12 180) (fields_autoplaced)
+  (global_label "GND" (shape output) (at 53.975 71.12 180) (fields_autoplaced)
     (effects (font (size 1.27 1.27)) (justify right))
     (property "Intersheetrefs" "${INTERSHEET_REFS}" (at 47.1193 71.12 0)
@@
     )
   )
-  (global_label "GND" (shape input) (at 53.975 73.66 180) (fields_autoplaced)
+  (global_label "GND" (shape output) (at 53.975 73.66 180) (fields_autoplaced)
     (effects (font (size 1.27 1.27)) (justify right))
     (property "Intersheetrefs" "${INTERSHEET_REFS}" (at 47.1193 73.66 0)
@@
     )
   )
-  (global_label "GND" (shape input) (at 53.975 60.96 180) (fields_autoplaced)
+  (global_label "GND" (shape output) (at 53.975 60.96 180) (fields_autoplaced)
     (effects (font (size 1.27 1.27)) (justify right))
     (property "Intersheetrefs" "${INTERSHEET_REFS}" (at 47.1193 60.96 0)
@@
     )
   )
-  (global_label "GND" (shape input) (at 53.975 81.28 180) (fields_autoplaced)
+  (global_label "GND" (shape output) (at 53.975 81.28 180) (fields_autoplaced)
     (effects (font (size 1.27 1.27)) (justify right))
     (property "Intersheetrefs" "${INTERSHEET_REFS}" (at 47.1193 81.28 0)

Commit message: some new parts
Parts:
- U3: footprint MQFN20_NU_MCH -> MCP9601:MQFN20_NU_MCH
Connections:
- no-connect marks 0 -> 4
Changed lines of the file:
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@@
   (junction (at 134.62 66.04) (diameter 0) (color 0 0 0 0)
   )
+  (no_connect (at 53.975 63.5))
+  (no_connect (at 53.975 55.88))
+  (no_connect (at 53.975 58.42))
+  (no_connect (at 53.975 66.04))
   (wire (pts (xy 116.84 81.915) (xy 116.84 78.74))
     (stroke (width 0) (type default))
@@
       (effects (font (size 1.524 1.524)))
     )
-    (property "Footprint" "MQFN20_NU_MCH" (at 106.045 85.344 0)
+    (property "Footprint" "MCP9601:MQFN20_NU_MCH" (at 106.045 85.344 0)
       (effects (font (size 1.27 1.27) italic) hide)
     )

Commit message: Todo notes after review
Parts:
- C7: value 0.1pF -> 0.1µF
Other:
- note added: "Werte nochmal anschauen"
Changed lines of the file:
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@@
     (stroke (width 0) (type default))
+  )
+  (text "Werte nochmal anschauen" (at 41.275 38.1 0)
+    (effects (font (size 1.27 1.27)) (justify left bottom))
   )
   (global_label "OCALERT" (shape output) (at 120.015 54.61 0) (fields_autoplaced)
@@
       (effects (font (size 1.27 1.27)) (justify left))
     )
-    (property "Value" "0.1pF" (at 119.38 77.4763 0)
+    (property "Value" "0.1µF" (at 119.38 77.4763 0)
       (effects (font (size 1.27 1.27)) (justify left))
     )

Commit message: first parts layout
Parts:
- R25: value 2MOhm -> 487 kOhm
- R27: value 1MOhm -> 2.49 MOhm
Other:
- note added: "Avionik fragen wegen TC"
- moved on the sheet: R25, TC1
Changed lines of the file:
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@@
     (stroke (width 0) (type default))
   )
-  (wire (pts (xy 116.84 78.74) (xy 125.095 78.74))
+  (wire (pts (xy 116.84 78.74) (xy 127 78.74))
     (stroke (width 0) (type default))
   )
@@
     (stroke (width 0) (type default))
   )
-  (wire (pts (xy 116.84 73.66) (xy 125.095 73.66))
+  (wire (pts (xy 116.84 73.66) (xy 127 73.66))
     (stroke (width 0) (type default))
   )
@@
     (stroke (width 0) (type default))
   )
-  (wire (pts (xy 125.095 71.12) (xy 127.635 71.12))
-    (stroke (width 0) (type default))
-  )
-  (wire (pts (xy 117.475 71.12) (xy 116.84 71.12))
+  (wire (pts (xy 132.715 71.12) (xy 142.24 71.12))
+    (stroke (width 0) (type default))
+  )
+  (wire (pts (xy 125.095 71.12) (xy 116.84 71.12))
     (stroke (width 0) (type default))
   )
@@
   (wire (pts (xy 139.065 46.355) (xy 155.575 46.355))
     (stroke (width 0) (type default))
+  )
+  (text "Avionik fragen wegen TC" (at 112.395 88.265 0)
+    (effects (font (size 1.27 1.27)) (justify left bottom))
   )
   (text "Werte nochmal anschauen" (at 41.275 38.1 0)
@@
     )
   )
-  (global_label "GND" (shape input) (at 127.635 71.12 0) (fields_autoplaced)
-    (effects (font (size 1.27 1.27)) (justify left))
-    (property "Intersheetrefs" "${INTERSHEET_REFS}" (at 134.4907 71.12 0)
+  (global_label "GND" (shape input) (at 142.24 71.12 0) (fields_autoplaced)
+    (effects (font (size 1.27 1.27)) (justify left))
+    (property "Intersheetrefs" "${INTERSHEET_REFS}" (at 149.0957 71.12 0)
       (effects (font (size 1.27 1.27)) (justify left) hide)
     )
@@
       (effects (font (size 1.27 1.27)))
     )
-    (property "Value" "1MOhm" (at 156.845 80.01 90)
+    (property "Value" "2.49 MOhm" (at 156.845 80.01 90)
       (effects (font (size 1.27 1.27)))
     )
@@
     )
   )
-  (symbol (lib_id "Device:Thermocouple") (at 127.635 76.2 180) (unit 1)
+  (symbol (lib_id "Device:Thermocouple") (at 129.54 76.2 180) (unit 1)
     (in_bom yes) (on_board yes) (dnp no) (fields_autoplaced)
-    (property "Reference" "TC1" (at 132.715 74.93 0)
+    (property "Reference" "TC1" (at 134.62 74.93 0)
       (effects (font (size 1.27 1.27)) (justify right))
     )
-    (property "Value" "Thermocouple" (at 132.715 77.47 0)
+    (property "Value" "Thermocouple" (at 134.62 77.47 0)
       (effects (font (size 1.27 1.27)) (justify right))
     )
-    (property "Footprint" "" (at 142.24 77.47 0)
-      (effects (font (size 1.27 1.27)) hide)
-    )
-    (property "Datasheet" "~" (at 142.24 77.47 0)
+    (property "Footprint" "" (at 144.145 77.47 0)
+      (effects (font (size 1.27 1.27)) hide)
+    )
+    (property "Datasheet" "~" (at 144.145 77.47 0)
       (effects (font (size 1.27 1.27)) hide)
     )
@@
     )
   )
-  (symbol (lib_id "Device:R") (at 121.285 71.12 90) (unit 1)
+  (symbol (lib_id "Device:R") (at 128.905 71.12 90) (unit 1)
     (in_bom yes) (on_board yes) (dnp no)
-    (property "Reference" "R25" (at 114.3 69.85 90)
-      (effects (font (size 1.27 1.27)))
-    )
-    (property "Value" "2MOhm" (at 114.3 71.755 90)
-      (effects (font (size 1.27 1.27)))
-    )
-    (property "Footprint" "" (at 121.285 72.898 90)
-      (effects (font (size 1.27 1.27)) hide)
-    )
-    (property "Datasheet" "~" (at 121.285 71.12 0)
-      (effects (font (size 1.27 1.27)) hide)
-    )
+    (property "Reference" "R25" (at 121.92 69.85 90)
+      (effects (font (size 1.27 1.27)))
+    )
+    (property "Value" "487 kOhm" (at 121.92 71.755 90)
+      (effects (font (size 1.27 1.27)))
+    )
+    (property "Footprint" "" (at 128.905 72.898 90)
+      (effects (font (size 1.27 1.27)) hide)
+    )
+    (property "Datasheet" "~" (at 128.905 71.12 0)
+      (effects (font (size 1.27 1.27)) hide)
+    )
