File: Payload_PCB/heating_pad.kicad_sch (KiCad schematic)
At the start: 6 parts, among them J6 Conn_01x02_Pin, Q30 SSM3K36TU,LF, U14 TSR_1-2450

Commit message: Added some actual parts
Parts:
- removed J6: Conn_01x02_Pin, symbol Connector:Conn_01x02_Pin
- added HeatingPadConnector1: 436500204, CON_436500204_MOL, symbol 436500204:436500204
Connections:
- net 0.5A: now also HeatingPadConnector1.2
- net at Q30.3 (D): now also HeatingPadConnector1.1
Other:
- note removed: "Connector to heating pad"
- company: (none) -> SpaceTeam Aachen
- title: (none) -> Heating Pad and Control
Changed lines of the file:
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@@
 (kicad_sch (version 20230121) (generator eeschema)
   (paper "A5")
+  (title_block
+    (title "Heating Pad and Control")
+    (company "SpaceTeam Aachen")
+  )
   (junction (at 144.145 76.835) (diameter 0) (color 0 0 0 0)
   )
@@
     (stroke (width 0) (type default))
   )
+  (wire (pts (xy 94.615 50.165) (xy 94.615 62.23))
+    (stroke (width 0) (type default))
+  )
   (wire (pts (xy 131.445 62.23) (xy 133.985 62.23))
     (stroke (width 0) (type default))
   )
-  (wire (pts (xy 104.775 62.23) (xy 117.475 62.23))
+  (wire (pts (xy 94.615 62.23) (xy 117.475 62.23))
     (stroke (width 0) (type default))
   )
@@
     (stroke (width 0) (type default))
   )
+  (wire (pts (xy 88.265 47.625) (xy 88.265 60.325))
+    (stroke (width 0) (type default))
+  )
   (wire (pts (xy 117.475 76.835) (xy 117.475 73.025))
     (stroke (width 0) (type default))
@@
     (stroke (width 0) (type default))
   )
-  (wire (pts (xy 104.775 62.23) (xy 104.775 52.705))
-    (stroke (width 0) (type default))
-  )
-  (wire (pts (xy 88.265 50.165) (xy 104.775 50.165))
+  (wire (pts (xy 88.265 47.625) (xy 107.315 47.625))
     (stroke (width 0) (type default))
   )
@@
     (stroke (width 0) (type default))
   )
-  (wire (pts (xy 88.265 60.325) (xy 88.265 50.165))
-    (stroke (width 0) (type default))
-  )
   (wire (pts (xy 88.265 86.995) (xy 88.265 90.805))
     (stroke (width 0) (type default))
@@
     (stroke (width 0) (type default))
   )
-  (text "Connector to \nheating pad\n" (at 105.41 46.99 0)
-    (effects (font (size 1.27 1.27)) (justify left bottom))
+  (wire (pts (xy 94.615 50.165) (xy 107.315 50.165))
+    (stroke (width 0) (type default))
   )
   (text "Switching frequency 500kHz" (at 119.38 64.77 0)
@@
         (path "/5c4f9a68-5778-4223-b18a-2e31db8d7d40/33b2e5d7-5e3f-425c-b4f0-5321d20d308b"
           (reference "R84") (unit 1)
-        )
-      )
-    )
-  )
-  (symbol (lib_id "Connector:Conn_01x02_Pin") (at 109.855 52.705 180) (unit 1)
-    (in_bom yes) (on_board yes) (dnp no)
-    (property "Reference" "J6" (at 111.76 50.165 0)
-      (effects (font (size 1.27 1.27)))
-    )
-    (property "Value" "Conn_01x02_Pin" (at 118.11 52.07 0)
-      (effects (font (size 1.27 1.27)))
-    )
-    (property "Footprint" "" (at 109.855 52.705 0)
-      (effects (font (size 1.27 1.27)) hide)
-    )
-    (property "Datasheet" "~" (at 109.855 52.705 0)
-      (effects (font (size 1.27 1.27)) hide)
-    )
-    (pin "1")
-    (pin "2")
-    (instances
-      (project "Payload_PCB"
-        (path "/5c4f9a68-5778-4223-b18a-2e31db8d7d40"
-          (reference "J6") (unit 1)
-        )
-        (path "/5c4f9a68-5778-4223-b18a-2e31db8d7d40/1e9e1733-6b5a-4028-9f43-052cd8d181d3"
-          (reference "J6") (unit 1)
-        )
-        (path "/5c4f9a68-5778-4223-b18a-2e31db8d7d40/d053929f-48bc-4e65-8bde-26e573685ab7"
-          (reference "J7") (unit 1)
-        )
-        (path "/5c4f9a68-5778-4223-b18a-2e31db8d7d40/33b2e5d7-5e3f-425c-b4f0-5321d20d308b"
-          (reference "J8") (unit 1)
         )
       )
@@
         )
       )
+    )
+  )
+  (symbol (lib_id "436500204:436500204") (at 107.315 47.625 0) (unit 1)
+    (in_bom yes) (on_board yes) (dnp no)
+    (property "Reference" "HeatingPadConnector1" (at 120.015 47.625 0)
+      (effects (font (size 1.524 1.524)) (justify left))
+    )
+    (property "Value" "436500204" (at 120.015 50.165 0)
+      (effects (font (size 1.524 1.524)) (justify left))
+    )
+    (property "Footprint" "CON_436500204_MOL" (at 107.315 47.625 0)
+      (effects (font (size 1.27 1.27) italic) hide)
+    )
+    (property "Datasheet" "436500204" (at 107.315 47.625 0)
+      (effects (font (size 1.27 1.27) italic) hide)
+    )
+    (pin "1")
+    (pin "2")
+    (pin "P1")
+    (pin "P2")
+    (instances
+      (project "Payload_PCB"
+        (path "/5c4f9a68-5778-4223-b18a-2e31db8d7d40/1e9e1733-6b5a-4028-9f43-052cd8d181d3"
+          (reference "HeatingPadConnector1") (unit 1)
+        )
+        (path "/5c4f9a68-5778-4223-b18a-2e31db8d7d40/d053929f-48bc-4e65-8bde-26e573685ab7"
+          (reference "HeatingPadConnector2") (unit 1)
+        )
+        (path "/5c4f9a68-5778-4223-b18a-2e31db8d7d40/33b2e5d7-5e3f-425c-b4f0-5321d20d308b"
+          (reference "HeatingPadConnector3") (unit 1)
+        )
+      )

Commit message: some new parts
Parts:
- Q30: footprint SOTFL65P210X75-3N -> footprints:SOTFL65P210X75-3N
Connections:
- no-connect marks 0 -> 2
Changed lines of the file:
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@@
   (junction (at 88.265 86.995) (diameter 0) (color 0 0 0 0)
   )
+  (no_connect (at 107.315 55.245))
+  (no_connect (at 107.315 52.705))
   (wire (pts (xy 117.475 76.835) (xy 144.145 76.835))
     (stroke (width 0) (type default))
@@
       (effects (font (size 1.27 1.27)) (justify left))
     )
-    (property "Footprint" "SOTFL65P210X75-3N" (at 92.075 169.215 0)
+    (property "Footprint" "footprints:SOTFL65P210X75-3N" (at 92.075 169.215 0)
       (effects (font (size 1.27 1.27)) (justify left top) hide)
     )

Commit message: Todo notes after review
Parts:
- R78: value 200 Ohm -> 10kOhm
Other:
- note added: "Filter überflüssig"
Changed lines of the file:
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@@
     (stroke (width 0) (type default))
+  )
+  (text "Filter überflüssig" (at 116.84 80.01 0)
+    (effects (font (size 1.27 1.27)) (justify left bottom))
   )
   (text "Switching frequency 500kHz" (at 119.38 64.77 0)
@@
       (effects (font (size 1.27 1.27)) (justify left))
     )
-    (property "Value" "200 Ohm" (at 74.295 81.915 0)
+    (property "Value" "10kOhm" (at 74.295 81.915 0)
       (effects (font (size 1.27 1.27)) (justify left))
     )

Commit message: first parts layout
Parts:
- removed C33: 10µF, symbol Device:C
- removed L3: 10µH, symbol Device:L
Connections:
- net 0.5A: now also U14.3 (Vout)
Changed lines of the file:
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@@
     (company "SpaceTeam Aachen")
   )
-  (junction (at 144.145 76.835) (diameter 0) (color 0 0 0 0)
-  )
   (junction (at 73.025 70.485) (diameter 0) (color 0 0 0 0)
-  )
-  (junction (at 117.475 62.23) (diameter 0) (color 0 0 0 0)
   )
   (junction (at 88.265 86.995) (diameter 0) (color 0 0 0 0)
@@
   (no_connect (at 107.315 55.245))
   (no_connect (at 107.315 52.705))
-  (wire (pts (xy 117.475 76.835) (xy 144.145 76.835))
-    (stroke (width 0) (type default))
-  )
   (wire (pts (xy 94.615 50.165) (xy 94.615 62.23))
     (stroke (width 0) (type default))
   )
-  (wire (pts (xy 131.445 62.23) (xy 133.985 62.23))
-    (stroke (width 0) (type default))
-  )
-  (wire (pts (xy 94.615 62.23) (xy 117.475 62.23))
+  (wire (pts (xy 94.615 62.23) (xy 133.985 62.23))
     (stroke (width 0) (type default))
   )
@@
     (stroke (width 0) (type default))
   )
-  (wire (pts (xy 117.475 76.835) (xy 117.475 73.025))
-    (stroke (width 0) (type default))
-  )
-  (wire (pts (xy 144.145 76.835) (xy 144.145 78.74))
+  (wire (pts (xy 144.145 69.85) (xy 144.145 78.74))
     (stroke (width 0) (type default))
   )
@@
     (stroke (width 0) (type default))
   )
-  (wire (pts (xy 117.475 62.23) (xy 123.825 62.23))
-    (stroke (width 0) (type default))
-  )
-  (wire (pts (xy 117.475 62.23) (xy 117.475 65.405))
-    (stroke (width 0) (type default))
-  )
   (wire (pts (xy 88.265 86.995) (xy 88.265 90.805))
     (stroke (width 0) (type default))
@@
     (stroke (width 0) (type default))
   )
-  (wire (pts (xy 144.145 69.85) (xy 144.145 76.835))
-    (stroke (width 0) (type default))
-  )
   (wire (pts (xy 73.025 70.485) (xy 80.645 70.485))
     (stroke (width 0) (type default))
@@
     (stroke (width 0) (type default))
   )
-  (text "Filter überflüssig" (at 116.84 80.01 0)
+  (text "Filter überflüssig" (at 117.475 65.405 0)
     (effects (font (size 1.27 1.27)) (justify left bottom))
   )
-  (text "Switching frequency 500kHz" (at 119.38 64.77 0)
+  (text "Switching frequency 500kHz" (at 146.05 69.85 0)
     (effects (font (size 0.762 0.762)) (justify left bottom))
   )
@@
         (path "/5c4f9a68-5778-4223-b18a-2e31db8d7d40/33b2e5d7-5e3f-425c-b4f0-5321d20d308b"
           (reference "Q38") (unit 1)
-        )
-      )
-    )
-  )
-  (symbol (lib_id "Device:C") (at 117.475 69.215 0) (unit 1)
-    (in_bom yes) (on_board yes) (dnp no)
-    (property "Reference" "C33" (at 120.65 67.945 0)
-      (effects (font (size 1.27 1.27)) (justify left))
-    )
-    (property "Value" "10µF" (at 120.65 70.485 0)
-      (effects (font (size 1.27 1.27)) (justify left))
-    )
-    (property "Footprint" "" (at 118.4402 73.025 0)
-      (effects (font (size 1.27 1.27)) hide)
-    )
-    (property "Datasheet" "~" (at 117.475 69.215 0)
-      (effects (font (size 1.27 1.27)) hide)
-    )
-    (pin "1")
-    (pin "2")
-    (instances
-      (project "Payload_PCB"
-        (path "/5c4f9a68-5778-4223-b18a-2e31db8d7d40/1e9e1733-6b5a-4028-9f43-052cd8d181d3"
-          (reference "C33") (unit 1)
-        )
-        (path "/5c4f9a68-5778-4223-b18a-2e31db8d7d40/d053929f-48bc-4e65-8bde-26e573685ab7"
-          (reference "C32") (unit 1)
-        )
-        (path "/5c4f9a68-5778-4223-b18a-2e31db8d7d40/33b2e5d7-5e3f-425c-b4f0-5321d20d308b"
-          (reference "C34") (unit 1)
         )
       )
@@
         )
       )
-    )
-  )
-  (symbol (lib_id "Device:L") (at 127.635 62.23 90) (unit 1)
-    (in_bom yes) (on_board yes) (dnp no)
-    (property "Reference" "L3" (at 127.635 58.42 90)
-      (effects (font (size 1.27 1.27)))
-    )
-    (property "Value" "10µH" (at 127.635 60.325 90)
-      (effects (font (size 1.27 1.27)))
-    )
-    (property "Footprint" "" (at 127.635 62.23 0)
-      (effects (font (size 1.27 1.27)) hide)
-    )
-    (property "Datasheet" "~" (at 127.635 62.23 0)
-      (effects (font (size 1.27 1.27)) hide)
-    )
-    (pin "1")
-    (pin "2")
-    (instances
-      (project "Payload_PCB"
-        (path "/5c4f9a68-5778-4223-b18a-2e31db8d7d40"
-          (reference "L3") (unit 1)
-        )
-        (path "/5c4f9a68-5778-4223-b18a-2e31db8d7d40/d053929f-48bc-4e65-8bde-26e573685ab7"
-          (reference "L3") (unit 1)
-        )
-        (path "/5c4f9a68-5778-4223-b18a-2e31db8d7d40/1e9e1733-6b5a-4028-9f43-052cd8d181d3"
-          (reference "L4") (unit 1)
-        )
-        (path "/5c4f9a68-5778-4223-b18a-2e31db8d7d40/33b2e5d7-5e3f-425c-b4f0-5321d20d308b"
-          (reference "L5") (unit 1)
-        )
-      )
