File: Payload_PCB/solenoid_control.kicad_sch (KiCad schematic)
At the start: 9 parts, among them Q28 SI1308EDL-T1-BE3, Q30 SSM3K36TU,LF, Q6 SI1308EDL-T1-BE3

Commit message: first parts layout
Parts:
- added D12, D3: D_Schottky, symbol Device:D_Schottky
Connections:
- net GND: now also D12.2 (A), D3.2 (A)
- net s_blue: now also D3.1 (K)
- net s_white: now also D12.1 (K)
Other:
- note added: "Freilaufdioden"
- note removed: "Diode zum entladen"
- moved on the sheet: C3, D6, Q28, Q30, Q6, R5, R6, R7, R77
