File: payload_externPressureSensor/payload_externPressureSensor.kicad_sch (KiCad schematic)
At the start: 6 parts, among them IC1 BMP390

Commit message: first parts layout
Other:
- note added: "1110110x"
- note removed: "1110110"
Changed lines of the file:
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@@
     (stroke (width 0) (type default))
   )
-  (text "1110110" (at 123.825 64.135 0)
+  (text "1110110x" (at 123.825 64.135 0)
     (effects (font (size 0.762 0.762)) (justify left bottom))
   )
